File: qmmister-sd-relocate.kicad_pcb (KiCad board)
At the start: 2 copper layers, 25 x 46.2 mm, 7 parts, among them J1 Micro_SD_Card_Det1, J2 Micro_SD_Card_Det1, J3 Conn_01x09, J4 Conn_01x09, J5 PinHeader_1x02_P2.54mm_Vertic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, J6 PinHeader_2x05_P2.54mm_Vertic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

Commit message: Minor tweaks - allow VSS pad to utilize fill zone
Connections:
- J2 pad 6: Net-(J2-VSS) -> GND
Changed lines of the file:
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@@
 			(size 0.7 1.6)
 			(layers "F.Cu" "F.Paste" "F.Mask")
-			(net 16 "Net-(J2-VSS)")
+			(net 19 "GND")
 			(pinfunction "VSS")
 			(pintype "power_in")
